Commit message: finish1：refactor(arm_urdf): 迁移ROS1项目至ROS2并修复关节控制问题
重构项目结构，将原ROS1的arm2.0包迁移为ROS2兼容的arm_urdf包。主要变更包括：
- 更新package.xml和CMakeLists.txt为ROS2格式
- 修复所有关节限制参数，解决GUI控制失效问题
- 新增ROS2风格的Python启动文件
- 添加详细文档说明和测试脚本

删除冗余的arm6包及其相关文件，包括：
- 旧的ROS1启动文件
- 重复的配置和网格文件
- 过时的测试脚本和批处理文件

File: arm_urdf/urdf/arm2.0.urdf (robot description, URDF)
Before this commit: robot arm2.0, 7 links, 6 joints
Links:
- link Link1: geometry collision mesh filename=package://arm_urdf/meshes/Link1.STL; visual mesh filename=package://arm_urdf/meshes/Link1.STL
- link Link2: geometry collision mesh filename=package://arm_urdf/meshes/Link2.STL; visual mesh filename=package://arm_urdf/meshes/Link2.STL
- link Link3: geometry collision mesh filename=package://arm_urdf/meshes/Link3.STL; visual mesh filename=package://arm_urdf/meshes/Link3.STL
- link Link4: geometry collision mesh filename=package://arm_urdf/meshes/Link4.STL; visual mesh filename=package://arm_urdf/meshes/Link4.STL
- link Link5: geometry collision mesh filename=package://arm_urdf/meshes/Link5.STL; visual mesh filename=package://arm_urdf/meshes/Link5.STL
- link Link6: geometry collision mesh filename=package://arm_urdf/meshes/Link6.STL; visual mesh filename=package://arm_urdf/meshes/Link6.STL
- link base_link: geometry collision mesh filename=package://arm_urdf/meshes/base_link.STL; visual mesh filename=package://arm_urdf/meshes/base_link.STL
Joints:
- joint j1: limit lower=0 upper=0 effort=0 velocity=0 -> lower=-3.14159 upper=3.14159 effort=100 velocity=2.0
- joint j2: limit lower=0 upper=0 effort=0 velocity=0 -> lower=-3.14159 upper=3.14159 effort=100 velocity=2.0
- joint j3: limit lower=0 upper=0 effort=0 velocity=0 -> lower=-3.14159 upper=3.14159 effort=100 velocity=2.0
- joint j4: limit lower=0 upper=0 effort=0 velocity=0 -> lower=-3.14159 upper=3.14159 effort=100 velocity=2.0
- joint j5: limit lower=0 upper=0 effort=0 velocity=0 -> lower=-3.14159 upper=3.14159 effort=100 velocity=2.0
- joint j6: limit lower=0 upper=0 effort=0 velocity=0 -> lower=-3.14159 upper=3.14159 effort=100 velocity=2.0
